File: cpu.sch (KiCad schematic (older format))
At the start: 46 parts, among them P1 GND, P513 TP1, P514 TP2, P515 TP3, P523 UART4, P542 TP4, P543 TP5, P545 TP7, P546 TP8, P547 TP9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

Commit message: [cleanup] updating project files for LEIA
Parts:
- D1, D2: symbol wookey:ZENERsmall -> leia:ZENERsmall
- D110, D111: symbol wookey:LED -> leia:LED
- SW503, SW514: footprint wookey:KSR_TACTILE_SWITCH -> leia:KSR_TACTILE_SWITCH; symbol wookey:SW_PUSH -> leia:SW_PUSH
- U1: symbol wookey:LD1117S33TR -> leia:LD1117S33TR
- U500: symbol wookey:STM32F417VE -> leia:STM32F417VE
Changed lines of the file:
@@
 EESchema Schematic File Version 4
-LIBS:wookey-cache
+LIBS:leia-cache
 EELAYER 29 0
 EELAYER END
@@
 $EndDescr
 $Comp
-L wookey:LD1117S33TR U1
+L leia:LD1117S33TR U1
 U 1 1 5CDD01A8
 P 4250 2950
@@
 $EndComp
 $Comp
-L wookey:GND #PWR0133
+L leia:GND #PWR0133
 U 1 1 5CDD01AC
 P 4250 3450
@@
 $EndComp
 $Comp
-L wookey:ZENERsmall D1
+L leia:ZENERsmall D1
 U 1 1 557FE9CE
 P 2550 2400
@@
 $EndComp
 $Comp
-L wookey:+3V3 #PWR0134
+L leia:+3V3 #PWR0134
 U 1 1 5CDD01AD
 P 5050 2900
@@
 $EndComp
 $Comp
-L wookey:GND #PWR0135
+L leia:GND #PWR0135
 U 1 1 557FEFE3
 P 1450 5600
@@
 $EndComp
 $Comp
-L wookey:+3V3 #PWR0136
+L leia:+3V3 #PWR0136
 U 1 1 557FF00F
 P 1450 4150
@@
 USB_HS_VBUS
 $Comp
-L wookey:LED D111
+L leia:LED D111
 U 1 1 557FF390
 P 3500 5450
@@
 $EndComp
 $Comp
-L wookey:LED D110
+L leia:LED D110
 U 1 1 557FF3FD
 P 3150 5450
@@
 LED1_PC5
 $Comp
-L wookey:+3V3 #PWR0137
+L leia:+3V3 #PWR0137
 U 1 1 5CDD01B1
 P 10600 3300
@@
 $EndComp
 $Comp
-L wookey:+3V3 #PWR0138
+L leia:+3V3 #PWR0138
 U 1 1 55801B5A
 P 10950 4850
@@
 $EndComp
 $Comp
-L wookey:GND #PWR0139
+L leia:GND #PWR0139
 U 1 1 55801C6D
 P 10300 4000
@@
 $EndComp
 $Comp
-L wookey:GND #PWR0140
+L leia:GND #PWR0140
 U 1 1 558023B8
 P 10650 11300
@@
 $EndComp
 $Comp
-L wookey:GND #PWR0141
+L leia:GND #PWR0141
 U 1 1 55802906
 P 11550 11650
@@
 $EndComp
 $Comp
-L wookey:GND #PWR0142
+L leia:GND #PWR0142
 U 1 1 558063EC
 P 7950 5750
@@
 $EndComp
 $Comp
-L wookey:+3V3 #PWR0143
+L leia:+3V3 #PWR0143
 U 1 1 5CDD01B8
 P 7950 4550
@@
 $EndComp
 $Comp
-L wookey:SW_PUSH SW514
+L leia:SW_PUSH SW514
 U 1 1 55806494
 P 7650 5400
 F 0 "SW514" H 7800 5510 50  0000 C CNN
 F 1 "RESET" H 7650 5320 50  0000 C CNN
-F 2 "wookey:KSR_TACTILE_SWITCH" H 7650 5400 60  0001 C CNN
+F 2 "leia:KSR_TACTILE_SWITCH" H 7650 5400 60  0001 C CNN
 F 3 "http://www.farnell.com/datasheets/1780692.pdf" H 7650 5400 60  0001 C CNN
 F 4 "C & K COMPONENTS" H 7650 5400 60  0001 C CNN "MFG Name"
@@
 $EndComp
 $Comp
-L wookey:+3V3 #PWR0145
+L leia:+3V3 #PWR0145
 U 1 1 5CDD01BA
 P 20350 2400
@@
 $EndComp
 $Comp
-L wookey:GND #PWR0146
+L leia:GND #PWR0146
 U 1 1 559EE3ED
 P 3300 5750
@@
 EXTENSION & DEBUG
 $Comp
-L wookey:GND #PWR0147
+L leia:GND #PWR0147
 U 1 1 55A4B025
 P 20150 5400
@@
 EXT_5V
 $Comp
-L wookey:+5V #PWR0148
+L leia:+5V #PWR0148
 U 1 1 5CDD01BD
 P 3500 2900
@@
 $EndComp
 $Comp
-L wookey:GND #PWR0149
+L leia:GND #PWR0149
 U 1 1 55B89A86
 P 20150 3800
@@
 $EndComp
 $Comp
-L wookey:+3V3 #PWR0150
+L leia:+3V3 #PWR0150
 U 1 1 583F464B
 P 18900 3750
@@
 NoConn ~ 9650 6500
 $Comp
-L wookey:ZENERsmall D2
+L leia:ZENERsmall D2
 U 1 1 58B9AE08
 P 2550 2650
@@
 $EndComp
 $Comp
-L wookey:SW_PUSH SW503
+L leia:SW_PUSH SW503
 U 1 1 58BDB2DF
 P 5200 4500
 F 0 "SW503" H 5350 4610 50  0000 C CNN
 F 1 "DFU" H 5200 4420 50  0000 C CNN
-F 2 "wookey:KSR_TACTILE_SWITCH" H 5200 4500 60  0001 C CNN
+F 2 "leia:KSR_TACTILE_SWITCH" H 5200 4500 60  0001 C CNN
 F 3 "http://www.farnell.com/datasheets/1780692.pdf" H 5200 4500 60  0001 C CNN
 F 4 "C & K COMPONENTS" H 5200 4500 60  0001 C CNN "MFG Name"
@@
 $EndComp
 $Comp
-L wookey:GND #PWR0151
+L leia:GND #PWR0151
 U 1 1 58BDB96C
 P 5200 5300
@@
 $EndComp
 $Comp
-L wookey:+3V3 #PWR0152
+L leia:+3V3 #PWR0152
 U 1 1 5CDD01C1
 P 5200 4100
@@
 DFU
 $Comp
-L wookey:STM32F417VE U500
+L leia:STM32F417VE U500
 U 1 1 555A55E3
 P 11150 8100
@@
 $EndComp
 $Comp
-L wookey:GND #PWR0153
+L leia:GND #PWR0153
 U 1 1 55B89BB1
 P 20150 4600
@@
 NoConn ~ 9650 8000
 $Comp
-L wookey:GND #PWR0144
+L leia:GND #PWR0144
 U 1 1 5CCE517D
 P 20350 3050
