File: cpu.sch (KiCad schematic (older format))
At the start: 46 parts, among them P1 GND, P513 TP1, P514 TP2, P515 TP3, P523 UART4, P542 TP4, P543 TP5, P545 TP7, P546 TP8, P547 TP9, P548 TP10, P572 DEBUG/PROG, P592 UART1, P595 I2C1_SCL, P596 I2C1_SDA, SW503 DFU, SW514 RESET, U1 LD1117S33TR, U500 STM32F439VIT6

Commit message: [enhancement] add new file for chipwhisperer interface:iface_ufo.sch
Parts:
- removed C2, C6: 10uF, Capacitor_Tantalum_SMD:CP_EIA-1608-08_AVX-J, symbol Device:CP_Small
- removed C4: 100nF, Capacitor_SMD:C_0603_1608Metric, symbol Device:C_Small
- removed D1, D2: STPS1L30A, Diode_SMD:D_SMA, symbol leia:ZENERsmall
- removed P1: GND, TestPoint:TestPoint_Pad_1.0x1.0mm, symbol Connector_Generic:Conn_01x01
- removed P513: TP1, TestPoint:TestPoint_Pad_1.0x1.0mm, symbol Connector_Generic:Conn_01x01
- removed P514: TP2, TestPoint:TestPoint_Pad_1.0x1.0mm, symbol Connector_Generic:Conn_01x01
- removed P515: TP3, TestPoint:TestPoint_Pad_1.0x1.0mm, symbol Connector_Generic:Conn_01x01
- removed P523: UART4, Pin_Headers:Pin_Header_Straight_1x03, symbol Connector_Generic:Conn_01x03
- removed P572: DEBUG/PROG, Pin_Headers:Pin_Header_Straight_1x05, symbol Connector_Generic:Conn_01x05
- removed P595: I2C1_SCL, TestPoint:TestPoint_Pad_1.0x1.0mm, symbol Connector_Generic:Conn_01x01
- removed P596: I2C1_SDA, TestPoint:TestPoint_Pad_1.0x1.0mm, symbol Connector_Generic:Conn_01x01
- removed R595, R596: 47K, Resistor_SMD:R_0603_1608Metric, symbol Device:R_Small
- removed U1: LD1117S33TR, Package_TO_SOT_SMD:SOT-223, symbol leia:LD1117S33TR
- added D112: VDD, LED_SMD:LED_0603_1608Metric_Castellated, symbol Device:LED_ALT
- added JP100: BOOT1, Connector_PinHeader_2.54mm:PinHeader_1x02_P2.54mm_Vertical, symbol Device:Jumper_NO_Small
- added JP101: BOOT0, Connector_PinHeader_2.54mm:PinHeader_1x02_P2.54mm_Vertical, symbol Device:Jumper_NO_Small
- added P593: SWD, Connector_PinHeader_2.54mm:PinHeader_1x05_P2.54mm_Vertical, symbol Connector_Generic:Conn_01x05
- added R112: 470, Resistor_SMD:R_0603_1608Metric, symbol Device:R_Small
- C500, C506, C511, C514, C519, C521, C522, C528, C550, C575: Distrib FARNELL -> Farnell; Distrib Link https://fr.farnell.com/avx/0603yc104jat2a/condensateur-0-1-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 -> https://fr.farnell.com/murata/grm188r71h104ka93d/condensate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; Distrib Name (none) -> Farnell; Distrib PN 1740612 -> 8820023; MFG Name AVX -> Murata; MFG Part Num 0603YC104JAT2A -> GRM188R71H104KA93D
- C549, C573: footprint Capacitor_Tantalum_SMD:CP_EIA-1608-08_AVX-J -> Capacitor_SMD:C_0603_1608Metric; Distrib FARNELL -> Farnell; Distrib Link https://fr.farnell.com/avx/tacl225m016xta/condensateur-2-2-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 -> http://fr.farnell.com/murata/grm188r61c225ke15d/condensateu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; Distrib Name (none) -> Farnell; Distrib PN 1135275 -> 1735526; MFG Name AVX -> Murata; MFG Part Num TACL225M016XTA -> GRM188R61C225KE15D
- D110, D111: symbol leia:LED -> Device:LED_ALT; Distrib FARNELL -> Farnell; Distrib Name (none) -> Farnell; MFG Name VISHAY -> Vishay
- P542, P543, P545, P546, P547, P548: footprint TestPoint:TestPoint_Pad_1.0x1.0mm -> TestPoint:TestPoint_Pad_D1.0mm
- P592: footprint Pin_Headers:Pin_Header_Straight_1x03 -> Connector_PinHeader_2.54mm:PinHeader_1x03_P2.54mm_Vertical; Distrib (none) -> Farnell; Distrib Link http://fr.rs-online.com/web/p/embases-de-circuit-imprime/36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 -> https://fr.farnell.com/molex/90120-0763/connect-header-3-vo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; Distrib Name (none) -> Farnell; Distrib PN 360-6437 -> 9733310; MFG Name MOLEX -> Molex; MFG Part Num 90121-0763 -> 90120-0763
- R100, R503, R514: Distrib FARNELL -> Farnell; Distrib Link https://fr.farnell.com/vishay/crcw060310k0fkeahp/res-couche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 -> (none); Distrib Name (none) -> Farnell; Distrib Part Num (none) -> 1738918
- R104, R110, R111: Distrib FARNELL -> Farnell; Distrib Link https://fr.farnell.com/vishay/crcw0603470rfkea/res-couche-e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 -> (none); Distrib Name (none) -> Farnell; Distrib PN 2122323 -> 1469815; Distrib Part Num (none) -> 1469815; MFG Name Vishay -> Vishay
- SW503, SW514: symbol leia:SW_PUSH -> Switch:SW_Push; Distrib FARNELL -> Farnell; Distrib Name (none) -> Farnell
- U500: footprint Housings_QFP:LQFP-100_14x14mm_Pitch0.5mm -> Package_QFP:TQFP-100_14x14mm_P0.5mm; symbol leia:STM32F417VE -> leia-rescue:STM32F417VE; Distrib FARNELL -> Farnell; Distrib Name (none) -> Farnell
Connections:
- net labels added: CARD_PWR_EN, CARD_~R~W, GNDD, RX, TCK, TMS, TRIGGER, TX, VDD
- net labels removed: +5V, CARD_POWER, EXT_5V, HS_GPIO_HARD_RESET, HS_ULPI_CLK_PA5, HS_ULPI_D0_PA3, HS_ULPI_D1_PB0, HS_ULPI_D2_PB1, HS_ULPI_D3_PB10, HS_ULPI_D4_PB11, HS_ULPI_D5_PB12, HS_ULPI_D6_PB13, HS_ULPI_D7_PB5, HS_ULPI_DIR_PC2, HS_ULPI_NXT_PC3, HS_ULPI_STP_PC0, I2C1_SCL_PB8, I2C1_SDA_PB9, LED0, LED1, SCREEN_~D~C, SD_CLK, SD_CMD, SD_D0, SD_D1, SD_D2, SD_D3, SD_D4, SD_D5, SD_D6, SD_D7, SPI_MISO, SPI_MOSI, SPI_SCK, TCK/SWCLK, TMS/SWIO, TOUCH_BUSY, TOUCH_IRQ, TP1, TP2, TP3, USB_HS_HARD_RESET, USB_HS_ULPI_CLK, USB_HS_ULPI_D0, USB_HS_ULPI_D1, USB_HS_ULPI_D2, USB_HS_ULPI_D3, USB_HS_ULPI_D4, USB_HS_ULPI_D5, USB_HS_ULPI_D6, USB_HS_ULPI_D7, USB_HS_ULPI_DIR, USB_HS_ULPI_NXT, USB_HS_ULPI_STP, USB_HS_VBUS, ~SCREEN_RESET, ~SD_RST, ~SPI_FLASH_CS, ~SPI_FONT_CS, ~SPI_SCREEN_CS, ~SPI_TOUCH_CS
- wire segments 220 -> 162
- no-connect marks 21 -> 55
Other:
- note added: "Since the READER and the Target have separated \npower domains, the reader JTAG and the Debug UART\nare not connected to the CW308 board."
- note removed: "POWER"
- moved on the sheet: C500, C506, C514, C519, C521, C522, C528, C550, C575, P592, R100, R104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
