File: leia.sch (KiCad schematic (older format))
At the start: 9 parts

Commit message: [enhancement] Adding rshunt
Changed lines of the file:
@@
 $Descr A3 16535 11693
 encoding utf-8
-Sheet 1 6
-Title "Wookey Motherboard"
-Date "2019-05-16"
+Sheet 1 4
+Title "LEIA Motherboard"
+Date "2019-06-05"
 Rev ""
 Comp "ANSSI"
@@
 $EndSheet
 $Sheet
-S 13000 4850 2200 2700
-U 5B19B666
-F0 "screen" 50
-F1 "screen.sch" 50
-F2 "SCREEN_RESET" I L 13000 5350 50
-F3 "SCREEN_~D~C" I L 13000 5450 50
-F4 "TOUCH_IRQ" O L 13000 6500 50
-F5 "TOUCH_BUSY" O L 13000 6600 50
-F6 "~SPI_SCREEN_CS" I L 13000 5550 50
-F7 "~SPI_FLASH_CS" I L 13000 6850 50
-F8 "~SPI_TOUCH_CS" I L 13000 6400 50
-F9 "~SPI_FONT_CS" I L 13000 7050 50
-F10 "SPI_MISO" O L 13000 5750 50
-F11 "SPI_MOSI" I L 13000 5850 50
-F12 "SPI_SCK" I L 13000 5950 50
-F13 "+3V3" U L 13000 5050 50
-F14 "GND" U L 13000 7300 50
-$EndSheet
-$Sheet
 S 1200 4850 4850 2700
 U 5B19B7B2
@@
 Wire Wire Line
 	6400 7250 6400 7900
-Wire Wire Line
-	11750 6850 13000 6850
-Wire Wire Line
-	11750 7050 13000 7050
-Wire Wire Line
-	11750 6600 13000 6600
-Wire Wire Line
-	11750 6500 13000 6500
-Wire Wire Line
-	11750 6400 13000 6400
-Wire Wire Line
-	11750 5950 13000 5950
-Wire Wire Line
-	11750 5550 13000 5550
-Wire Wire Line
-	11750 5450 13000 5450
-Wire Wire Line
-	11750 5350 13000 5350
-Wire Wire Line
-	13000 5050 12700 5050
-Wire Wire Line
-	12700 5050 12700 4950
-Wire Wire Line
-	13000 7300 12700 7300
-Wire Wire Line
-	12700 7300 12700 7800
-Wire Wire Line
-	13000 4150 12700 4150
-Wire Wire Line
-	12700 4150 12700 4400
-Wire Wire Line
-	11750 2600 13000 2600
-Wire Wire Line
-	11750 2700 13000 2700
-Wire Wire Line
-	11750 2800 13000 2800
-Wire Wire Line
-	11750 2900 13000 2900
-Wire Wire Line
-	11750 2350 13000 2350
-Wire Wire Line
-	11750 2250 13000 2250
 $Comp
 L power:GND #PWR0101
@@
 $EndComp
 $Comp
-L power:GND #PWR0103
-U 1 1 5B2DDDEF
-P 12700 7800
-F 0 "#PWR0103" H 12700 7550 50  0001 C CNN
-F 1 "GND" H 12705 7627 50  0000 C CNN
-F 2 "" H 12700 7800 50  0001 C CNN
-F 3 "" H 12700 7800 50  0001 C CNN
-	1    12700 7800
-	1    0    0    -1
-$EndComp
-$Comp
-L power:GND #PWR0104
-U 1 1 5B2DDEC9
-P 12700 4400
-F 0 "#PWR0104" H 12700 4150 50  0001 C CNN
-F 1 "GND" H 12705 4227 50  0000 C CNN
-F 2 "" H 12700 4400 50  0001 C CNN
-F 3 "" H 12700 4400 50  0001 C CNN
-	1    12700 4400
-	1    0    0    -1
-$EndComp
-$Comp
 L power:GND #PWR0105
 U 1 1 5B2DE00B
@@
 $EndComp
 $Comp
-L power:+3.3V #PWR0107
-U 1 1 5B2DE0EF
-P 12700 4950
-F 0 "#PWR0107" H 12700 4800 50  0001 C CNN
-F 1 "+3.3V" H 12715 5123 50  0000 C CNN
-F 2 "" H 12700 4950 50  0001 C CNN
-F 3 "" H 12700 4950 50  0001 C CNN
-	1    12700 4950
-	1    0    0    -1
-$EndComp
-$Comp
 L power:+3.3V #PWR0108
 U 1 1 5B2E0BAC
@@
 	7900 1550 7900 1200
 Wire Wire Line
-	11750 5750 13000 5750
-Wire Wire Line
-	11750 5850 13000 5850
-Wire Wire Line
 	6050 2400 8150 2400
 Wire Wire Line
@@
 NoConn ~ 11750 3000
 NoConn ~ 11750 2050
-$Comp
-L power:+3.3V #PWR0106
-U 1 1 5B2DE056
-P 12750 1200
-F 0 "#PWR0106" H 12750 1050 50  0001 C CNN
-F 1 "+3.3V" H 12765 1373 50  0000 C CNN
-F 2 "" H 12750 1200 50  0001 C CNN
-F 3 "" H 12750 1200 50  0001 C CNN
-	1    12750 1200
-	1    0    0    -1
-$EndComp
-Wire Wire Line
-	13000 1550 12750 1550
-Wire Wire Line
-	12750 1550 12750 1200
 $Sheet
 S 8150 1400 3600 8950
@@
 F48 "~SD_RST" O R 11750 2050 50
 $EndSheet
-Wire Wire Line
-	11750 3300 12400 3300
-Wire Wire Line
-	12400 3300 12400 3400
-Wire Wire Line
-	12400 3400 13000 3400
-$Sheet
-S 13000 1350 2200 3050
-U 5B00AAC9
-F0 "storage" 50
-F1 "storage.sch" 50
-F2 "SD_CLK" I L 13000 2250 50
-F3 "SD_CMD" I L 13000 2350 50
-F4 "SD_D0" B L 13000 2600 50
-F5 "SD_D1" B L 13000 2700 50
-F6 "SD_D2" B L 13000 2800 50
-F7 "SD_D3" B L 13000 2900 50
-F8 "+3V3" U L 13000 1550 50
-F9 "GND" U L 13000 4150 50
-F10 "SD_SW" O L 13000 3400 50
-$EndSheet
-$Comp
+$Comp
