File: leia.sch (KiCad schematic (older format))
At the start: 9 parts

Commit message: [enhancement] add new file for chipwhisperer interface:iface_ufo.sch
Parts:
- removed FID2, FID3: FIDUCIAL, Fiducials:Fiducial_1mm_Dia_2.54mm_Outer_CopperTop, symbol Mechanical:Fiducial
- removed FID4, FID5, FID6: FIDUCIAL, Fiducials:Fiducial_1mm_Dia_2.54mm_Outer_CopperBottom, symbol Mechanical:Fiducial
- removed H3: H3, Mounting_Holes:MountingHole_2.2mm_M2_ISO14580_Pad, symbol Mechanical:MountingHole_Pad
- added C1003, C4004: 0.1uF 35V Tant, Capacitor_Tantalum_SMD:CP_EIA-3216-18_Kemet-A, symbol Device:CP_Small
- added FID1002, FID1003, FID1004, FID1005, FID1006: FIDUCIAL-RESCUE-rescue, Fiducial:Fiducial_1mm_Mask2mm, symbol leia:Mechanical_Fiducial
- added J1002: READER_GND, Connector_PinHeader_2.54mm:PinHeader_2x03_P2.54mm_Vertical, symbol Connector_Generic:Conn_02x03_Odd_Even
- added J1003: READER_VDD, Connector_PinHeader_2.54mm:PinHeader_2x03_P2.54mm_Vertical, symbol Connector_Generic:Conn_02x03_Odd_Even
- added J1101: TARGET_PWR, Connector_PinHeader_2.54mm:PinHeader_2x03_P2.54mm_Vertical, symbol Connector_Generic:Conn_02x03_Odd_Even
- added J1102: TARGET_GND, Connector_PinHeader_2.54mm:PinHeader_2x03_P2.54mm_Vertical, symbol Connector_Generic:Conn_02x03_Odd_Even
- added J1103: TARGET_EXT_PWR, Connector_Coaxial:SMA_Amphenol_132289_EdgeMount, symbol Connector:Conn_Coaxial
- added J1112: TARGET_SHUNT, Connector_Coaxial:SMA_Amphenol_132289_EdgeMount, symbol Connector:Conn_Coaxial
- added J6: EXT_READER_VCC, Connector_Coaxial:SMA_Amphenol_132289_EdgeMount, symbol Connector:Conn_Coaxial
- added JP1102: SHUNT Bypass, Connector_PinHeader_2.54mm:PinHeader_1x02_P2.54mm_Vertical, symbol Device:Jumper_NO_Small
- added P523: CMD, Connector_PinHeader_2.54mm:PinHeader_2x04_P2.54mm_Vertical, symbol Connector_Generic:Conn_02x04_Odd_Even
- added R1112: 0.1 1%, Resistor_SMD:R_0603_1608Metric, symbol Device:R_Small
- added TP1001: VDDD, TestPoint_Keystone_5000-5004_Miniature, symbol Connector:TestPoint_Alt
- added TP1002: DGND, TestPoint_Keystone_5000-5004_Miniature, symbol Connector:TestPoint_Alt
- added TP1101: VDDA, TestPoint:TestPoint_Pad_D1.0mm, symbol Connector:TestPoint
- added TP1112: GNDA, TestPoint:TestPoint_Pad_D1.0mm, symbol Connector:TestPoint
- added TP5001: VDDA, TestPoint_Keystone_5000-5004_Miniature, symbol Connector:TestPoint_Alt
- added TP5002: GNDA, TestPoint_Keystone_5000-5004_Miniature, symbol Connector:TestPoint_Alt
- added U520: FOD8012A, Package_SO:SOIC-8_3.9x4.9mm_P1.27mm, symbol optos:FOD8012A
- FID1001: renamed from FID1; value FIDUCIAL -> FIDUCIAL-RESCUE-rescue; footprint Fiducials:Fiducial_1mm_Dia_2.54mm_Outer_CopperTop -> Fiducial:Fiducial_1mm_Mask2mm; symbol Mechanical:Fiducial -> leia:Mechanical_Fiducial
- HOLE1: renamed from H1; value H1 -> HOLE; footprint Mounting_Holes:MountingHole_2.2mm_M2_ISO14580_Pad -> MountingHole:MountingHole_2.2mm_M2_ISO14580_Pad; symbol Mechanical:MountingHole_Pad -> Connector:TestPoint
- HOLE2: renamed from H2; value H2 -> HOLE; footprint Mounting_Holes:MountingHole_2.2mm_M2_ISO14580_Pad -> MountingHole:MountingHole_2.2mm_M2_ISO14580_Pad; symbol Mechanical:MountingHole_Pad -> Connector:TestPoint
Connections:
- net GND: no longer names the net of HOLE1.1
- net GND: no longer HOLE2.1
- new net: J1101.6 (Pin_6), J1103.1 (In)
- new net: J1102.6 (Pin_6), J1103.2 (Ext)
- new net CW_GND: J1102.2 (Pin_2)
- new net CW_PWR: J1101.2 (Pin_2)
- new net EXT_READER_GND: J1002.6 (Pin_6), J6.2 (Ext)
- new net EXT_READER_VCC: J1003.5 (Pin_5), J6.1 (In)
- new net GNDA: J1102.1 (Pin_1), J1102.3 (Pin_3), J1102.5 (Pin_5), J1112.2 (Ext), JP1102.2, P523.8 (Pin_8), R1112.2, TP1112.1, TP5002.1
- new net GNDCARD: J1112.1 (In), JP1102.1, R1112.1
- new net GNDD: C4004.2, J1002.1 (Pin_1), J1002.3 (Pin_3), J1002.5 (Pin_5), TP1002.1, U520.4 (GND1)
- new net GND_CONSOLE: C1003.2, P523.7 (Pin_7), U520.5 (GND2)
- new net RX_CMD: U520.2 (VOA)
- new net RX_CONSOLE: P523.3 (Pin_3), U520.7 (VINA)
- new net TX_CMD: U520.3 (VINB)
- new net TX_CONSOLE: P523.5 (Pin_5), U520.6 (VOB)
- new net USB_READER_GND: J1002.2 (Pin_2)
- new net USB_READER_VCC: J1003.1 (Pin_1)
- new net VDD: C4004.1, J1003.2 (Pin_2), J1003.4 (Pin_4), J1003.6 (Pin_6), TP1001.1, U520.1 (VDD1)
- new net VDDA: J1101.1 (Pin_1), J1101.3 (Pin_3), J1101.5 (Pin_5), P523.2 (Pin_2), TP1101.1, TP5001.1
- new net VDD_CONSOLE: C1003.1, P523.1 (Pin_1), U520.8 (VDD2)
- new net iface_ufo/RX: P523.6 (Pin_6)
- new net iface_ufo/TX: P523.4 (Pin_4)
- no-connect marks 4 -> 7
Other:
- note added: "JMP 1101 VDDA\n 1-2 CW-POWER\n 5-6 EXT-POWER\n"
- note added: "JMP 1102 GNDA\n 1-2 CW-GND\n 5-6 EXT-GND\n"
- note added: "Since LEIA embed an SMA for the shunt resistor,\nwe do not need to connect SHUNT signal to the \nCW308 board"
- note added: "User can choose between external \npower supply or CW power supply."
- note added: "User can choose to connect the CMD Console\nto the CW or something else. In this case optocoupler\npower supply should be provided by the device connected\nto the CMD Console."
- note added: "VDDD and GNDD are connected to \noptocouplers reader side"
- moved on the sheet: HOLE1, HOLE2
