File: usb.sch (KiCad schematic (older format))
At the start: 20 parts, among them P3000 USB_FS_OTG, P6000 USB_FS_OTG, P828 XI, U300 USBLC6-2, U600 USBLC6-2, U800 USB3300, Y2 ASEMB-24.000MHZ-LY-T

Commit message: [cleanup] updating project files for LEIA
Parts:
- P3000, P6000: footprint wookey:USB_Micro-B-MOLEX_105017-0001 -> leia:USB_Micro-B-MOLEX_105017-0001; symbol wookey:USB_OTG -> leia:USB_OTG
- U300, U600: symbol wookey:USBLC6-2 -> leia:USBLC6-2
- U800: symbol wookey:USB3300 -> leia:USB3300
- Y2: symbol wookey:ASE-xxxMHz-Oscillator -> leia:ASE-xxxMHz-Oscillator
Changed lines of the file:
@@
 EESchema Schematic File Version 4
-LIBS:wookey-cache
+LIBS:leia-cache
 EELAYER 29 0
 EELAYER END
@@
 $EndDescr
 $Comp
-L wookey:USB_OTG P3000
+L leia:USB_OTG P3000
 U 1 1 5589C2A1
 P 5900 9250
 F 0 "P3000" V 6200 9200 50  0000 C CNN
 F 1 "USB_FS_OTG" H 5900 9450 50  0000 C CNN
-F 2 "wookey:USB_Micro-B-MOLEX_105017-0001" V 5850 9150 60  0001 C CNN
+F 2 "leia:USB_Micro-B-MOLEX_105017-0001" V 5850 9150 60  0001 C CNN
 F 3 "http://www.molex.com/pdm_docs/sd/1050170001_sd.pdf" V 5850 9150 60  0001 C CNN
 F 4 "MOLEX" H 5900 9250 60  0001 C CNN "MFG Name"
@@
 $EndComp
 $Comp
-L wookey:+3V3 #PWR0111
+L leia:+3V3 #PWR0111
 U 1 1 5589C2A9
 P 15000 8600
@@
 $EndComp
 $Comp
-L wookey:USBLC6-2 U600
+L leia:USBLC6-2 U600
 U 1 1 5589C2B7
 P 8300 4900
@@
 $EndComp
 $Comp
-L wookey:USBLC6-2 U300
+L leia:USBLC6-2 U300
 U 1 1 5589C2B8
 P 7500 8800
@@
 $EndComp
 $Comp
-L wookey:+3V3 #PWR0112
+L leia:+3V3 #PWR0112
 U 1 1 5589C2CA
 P 14200 10400
@@
 USB_HS_CON_D+
 $Comp
-L wookey:GND #PWR0113
+L leia:GND #PWR0113
 U 1 1 55B6A459
 P 6000 4400
@@
 $EndComp
 $Comp
-L wookey:GND #PWR0114
+L leia:GND #PWR0114
 U 1 1 55BA9623
 P 6050 8250
@@
 $EndComp
 $Comp
-L wookey:GND #PWR0115
+L leia:GND #PWR0115
 U 1 1 55BAC01A
 P 14200 11100
@@
 $EndComp
 $Comp
-L wookey:GND #PWR0116
+L leia:GND #PWR0116
 U 1 1 55BAC5A7
 P 15100 11100
@@
 $EndComp
 $Comp
-L wookey:GND #PWR0117
+L leia:GND #PWR0117
 U 1 1 55BAC6CC
 P 11950 10400
@@
 $EndComp
 $Comp
-L wookey:GND #PWR0119
+L leia:GND #PWR0119
 U 1 1 55BACFB6
 P 17400 9250
@@
 $EndComp
 $Comp
-L wookey:GND #PWR0120
+L leia:GND #PWR0120
 U 1 1 55BAD543
 P 16800 9250
@@
 $EndComp
 $Comp
-L wookey:GND #PWR0121
+L leia:GND #PWR0121
 U 1 1 55BAD668
 P 16150 8800
@@
 ear
 $Comp
-L wookey:USB_OTG P6000
+L leia:USB_OTG P6000
 U 1 1 58A45C1E
 P 5850 5450
 F 0 "P6000" V 6150 5400 50  0000 C CNN
 F 1 "USB_FS_OTG" H 5850 5650 50  0000 C CNN
-F 2 "wookey:USB_Micro-B-MOLEX_105017-0001" V 5800 5350 60  0001 C CNN
+F 2 "leia:USB_Micro-B-MOLEX_105017-0001" V 5800 5350 60  0001 C CNN
 F 3 "http://www.molex.com/pdm_docs/sd/1050170001_sd.pdf" V 5800 5350 60  0001 C CNN
 F 4 "MOLEX" H 5850 5450 60  0001 C CNN "MFG Name"
@@
 	6050 8200 6250 8200
 $Comp
-L wookey:USB3300 U800
+L leia:USB3300 U800
 U 1 1 5589C2C1
 P 15100 9900
@@
 	8150 9450 10600 9450
 $Comp
-L wookey:+3V3 #PWR0122
+L leia:+3V3 #PWR0122
 U 1 1 5B0CCB6A
 P 18750 9000
@@
 $EndComp
 $Comp
-L wookey:GND #PWR0123
+L leia:GND #PWR0123
 U 1 1 5B0CCC51
 P 18750 9200
@@
 GND
 $Comp
-L wookey:ASE-xxxMHz-Oscillator Y2
+L leia:ASE-xxxMHz-Oscillator Y2
 U 1 1 5B9F8C34
 P 12400 9900
@@
 	13000 9900 12700 9900
 $Comp
-L wookey:+3V3 #PWR0118
+L leia:+3V3 #PWR0118
 U 1 1 5BB413A1
 P 12000 9350
