File: usb.sch (KiCad schematic (older format))
At the start: 20 parts, among them P3000 USB_FS_OTG, P6000 USB_FS_OTG, P828 XI, U300 USBLC6-2, U600 USBLC6-2, U800 USB3300, Y2 ASEMB-24.000MHZ-LY-T

Commit message: [enhancement] add new file for chipwhisperer interface:iface_ufo.sch
Parts:
- removed C201: 4.7uF, Capacitor_Tantalum_SMD:CP_EIA-1608-08_AVX-J, symbol Device:CP_Small
- removed C305, C806, C816, C825, C826, C829, C830: 100nF, Capacitor_SMD:C_0603_1608Metric, symbol Device:C_Small
- removed C815, C8292: 4.7uF, Capacitor_Tantalum_SMD:CP_EIA-1608-08_AVX-J, symbol Device:C_Small
- removed C828: 0.01uF, Capacitor_SMD:C_0603_1608Metric, symbol Device:C_Small
- removed P3000: USB_FS_OTG, leia:USB_Micro-B-MOLEX_105017-0001, symbol leia:USB_OTG
- removed P828: XI, Measurement_Points:Measurement_Point_Round-SMD-Pad_Small, symbol Connector_Generic:Conn_01x01
- removed R832: 12K [1%], Resistor_SMD:R_0603_1608Metric, symbol Device:R_Small
- removed U300: USBLC6-2, Package_TO_SOT_SMD:TSOT-23-6, symbol leia:USBLC6-2
- removed U800: USB3300, Package_DFN_QFN:QFN-32-1EP_5x5mm_P0.5mm_EP3.1x3.1mm_ThermalVias, symbol leia:USB3300
- removed Y2: ASEMB-24.000MHZ-LY-T, Oscillator:Oscillator_SMD_Abracon_ASE-4Pin_3.2x2.5mm, symbol leia:ASE-xxxMHz-Oscillator
- added C4001, C4003: 10uF, Capacitor_Tantalum_SMD:CP_EIA-3216-18_Kemet-A, symbol Device:CP_Small
- added C4002: 100nF, Capacitor_SMD:C_0603_1608Metric, symbol Device:C_Small
- added U4001: LD1117S33TR, Package_TO_SOT_SMD:SOT-223, symbol leia-rescue:LD1117S33TR
- C605: Distrib FARNELL -> Farnell; Distrib Link https://fr.farnell.com/avx/0603yc104jat2a/condensateur-0-1-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 -> https://fr.farnell.com/murata/grm188r71h104ka93d/condensate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; Distrib Name (none) -> Farnell; Distrib PN 1740612 -> 8820023; MFG Name AVX -> Murata; MFG Part Num 0603YC104JAT2A -> GRM188R71H104KA93D
- P6000: value USB_FS_OTG -> USB_FS; symbol leia:USB_OTG -> Connector:USB_OTG; Distrib FARNELL -> Farnell; Distrib Name (none) -> Farnell; MFG Name MOLEX -> Molex
- U600: footprint Package_TO_SOT_SMD:TSOT-23-6 -> Package_TO_SOT_SMD:SOT-23-6; symbol leia:USBLC6-2 -> leia-rescue:USBLC6-2; Distrib FARNELL -> Farnell; Distrib Link https://fr.farnell.com/stmicroelectronics/usblc6-2sc6/esd-p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 -> http://fr.farnell.com/stmicroelectronics/usblc6-2sc6/esd-pr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; Distrib Name (none) -> Farnell
Connections:
- net +3V3: now also C4003.1, U4001.2 (VO)
- net USB_FS_VBUS: now also C4001.1, C4002.1, U4001.3 (VI)
- net GND renamed GNDPWR
- net GNDPWR: now also C4001.2, C4002.2, C4003.2, U4001.1 (GND)
- no-connect marks 6 -> 1
Other:
- note added: "FIXME DUAL POWER\n"
- note added: "POWER"
- note removed: "Optional active high transceiver reset. \nThis is the same as a write to the ULPI Reset, \naddress 04h, bit 5. This does not reset the ULPI \nregister set. This pin includes an integrated pull-down \nresistor to ground. If not used, this pin can be floated \nor connected to ground (recommended)."
- note removed: "USB HIGH SPEED"
- note removed: "see qtzcry-app-notes.pdf (in datasheets)"
- moved on the sheet: C605
