File: smartcard.sch (KiCad schematic (older format))
At the start: 5 parts, among them P1000 ISO7816_NO

Commit message: [enhancement] add new file for chipwhisperer interface:iface_ufo.sch
Parts:
- removed R1002: 10, Resistor_SMD:R_0603_1608Metric, symbol Device:R_Small
- added C1101, C1108, C1201, C1208, C1301, C1308, C1401, C1408, C1501, C1508, C1601, C1608, C1701, C1708, C1801, C1806, C1902, C5001, C5002, C5003: 0.1uF 35V Tant, Capacitor_Tantalum_SMD:CP_EIA-3216-18_Kemet-A, symbol Device:CP_Small
- added D3001: VDDA, LED_SMD:LED_0603_1608Metric_Castellated, symbol Device:LED_ALT
- added J1001: FILTER, Connector_PinHeader_2.54mm:PinHeader_2x03_P2.54mm_Vertical, symbol Connector_Generic:Conn_02x03_Odd_Even
- added J1706: TARGET_TRIG, Connector_Coaxial:SMA_Amphenol_132289_EdgeMount, symbol Connector:Conn_Coaxial
- added JP1500: TEARING, Connector_PinHeader_2.54mm:PinHeader_1x02_P2.54mm_Vertical, symbol Device:Jumper_NC_Small
- added Q5001, Q5002: BSS84, Package_TO_SOT_SMD:SOT-23, symbol Transistor_FET:BSS84
- added R1007, R1422, R1902: 22k, Resistor_SMD:R_0603_1608Metric, symbol Device:R_Small
- added R1306, R1506: 10k, Resistor_SMD:R_0603_1608Metric, symbol Device:R_Small
- added R3001: 470, Resistor_SMD:R_0603_1608Metric, symbol Device:R_Small
- added R5002, R5003: DNP, Resistor_SMD:R_0603_1608Metric, symbol Device:R_Small
- added U1100, U1200, U1300, U1400, U1500, U1600, U1700, U1800, U5001: FOD8001, Package_SO:SOIC-8_3.9x4.9mm_P1.27mm, symbol optos:FOD8001
- added U1900, U5002: ADG719-EP, Package_TO_SOT_SMD:TSOT-23-6, symbol mux:ADG719-EP
- C1001: footprint Capacitor_Tantalum_SMD:CP_EIA-1608-08_AVX-J -> Capacitor_SMD:C_0603_1608Metric; Distrib FARNELL -> Farnell; Distrib Link https://fr.farnell.com/avx/f981a106mma/condensateur-10-f-10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 -> http://fr.farnell.com/vishay/tp8m106m6r3c/condensateur-tant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; Distrib Name (none) -> Farnell; Distrib PN 2747667 -> 2425568; MFG Name AVX -> Vishay; MFG Part Num F981A106MMA -> TP8M106M6R3C
- C1002: Distrib FARNELL -> Farnell; Distrib Link https://fr.farnell.com/avx/0603yc104jat2a/condensateur-0-1-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 -> https://fr.farnell.com/murata/grm188r71h104ka93d/condensate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; Distrib Name (none) -> Farnell; Distrib PN 1740612 -> 8820023; MFG Name AVX -> Murata; MFG Part Num 0603YC104JAT2A -> GRM188R71H104KA93D
- P1000: Distrib Name (none) -> RS
- R1001: value 10K -> 20k; Distrib FARNELL -> Farnell; Distrib Link https://fr.farnell.com/vishay/crcw060310k0fkeahp/res-couche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 -> (none); Distrib Name (none) -> Farnell; Distrib PN 1738918 -> 2616587; MFG Part Num CRCW060310K0FKEAHP -> RCA060320K0FKEA
Connections:
- net CARD_CLK: now also U1200.2 (Vin); no longer P1000.C3 (CLK)
- net CARD_CT: now also U1600.6 (Vout); no longer P1000.SW1, R1001.2
- net CARD_IO: now also U1900.5 (D); no longer P1000.C7 (I/O)
- net CARD_RESET: now also U1100.2 (Vin); no longer P1000.C2 (RST)
- net CARD_VPP: now also U1300.2 (Vin); no longer P1000.C6 (VPP)
- net SHUNT_L: now reaches P1000.C5 (GND)
- net +3V3 renamed VDDA
- net VDDA: now also C1108.1, C1208.1, C1308.1, C1408.1, C1508.1, C1608.1, C1708.1, C1801.1, C5002.1, C5003.1, Q5001.2 (S), Q5002.2 (S), R1007.1, R3001.1, R5002.1, R5003.1, U1100.8 (VDD2), U1200.8 (VDD2), U1300.8 (VDD2), U1400.8 (VDD2), U1500.8 (VDD2), U1600.1 (VDD1), U1700.8 (VDD2), U1800.1 (VDD1), U5001.8 (VDD2), U5002.2 (VDD)
- net CARD_POWER: no longer names the net of C1001.1, C1002.1
- net CARD_POWER: now also J1001.2 (Pin_2), J1001.4 (Pin_4), J1001.6 (Pin_6); no longer P1000.C1 (VCC)
- net GND renamed GNDA
- net GNDA: now also C1108.2, C1208.2, C1308.2, C1408.2, C1508.2, C1608.2, C1708.2, C1801.2, C5002.2, C5003.2, D3001.1 (K), J1001.5 (Pin_5), J1706.2 (Ext), R1306.2, R1506.2, U1100.5 (GND2), U1200.5 (GND2), U1300.5 (GND2), U1400.5 (GND2), U1500.5 (GND2), U1600.4 (GND1), U1700.5 (GND2), U1800.4 (GND1), U5001.5 (GND2), U5002.3 (GND)
- new net: Q5001.1 (G), U1300.6 (Vout)
- new net: R5002.2, U1400.6 (Vout), U5002.6 (S2)
- new net: JP1500.1, U1500.6 (Vout)
- new net: R5003.2, U1800.2 (Vin), U5002.4 (S1)
- new net: U5001.6 (Vout), U5002.1 (IN)
- new net: JP1500.2, Q5002.1 (G)
- new net: D3001.2 (A), R3001.2
- new net CARD_PWR_EN: U1500.2 (Vin)
- new net CARD_~R~W: U1900.1 (IN), U5001.2 (Vin)
- new net CRD_CLK: P1000.C3 (CLK), U1200.6 (Vout)
- new net CRD_CT: P1000.SW1, R1001.2, U1600.2 (Vin)
- new net CRD_IO: P1000.C7 (I/O), R1007.2, U5002.5 (D)
- new net CRD_PWR: J1001.1 (Pin_1), P1000.C1 (VCC), Q5002.3 (D), R1506.1
- new net CRD_RST: P1000.C2 (RST), U1100.6 (Vout)
- new net CRD_VPP: P1000.C6 (VPP), Q5001.3 (D), R1306.1
- new net GNDD: C1101.2, C1201.2, C1301.2, C1401.2, C1501.2, C1601.2, C1701.2, C1806.2, C1902.2, C5001.2, U1100.4 (GND1), U1200.4 (GND1), U1300.4 (GND1), U1400.4 (GND1), U1500.4 (GND1), U1600.5 (GND2), U1700.4 (GND1), U1800.5 (GND2), U1900.3 (GND), U5001.4 (GND1)
- new net IO_IN: R1422.2, U1400.2 (Vin), U1900.6 (S2)
- new net IO_OUT: R1902.2, U1800.6 (Vout), U1900.4 (S1)
- new net TRIGGER: U1700.2 (Vin)
- new net TRIGGER_OUT: J1706.1 (In), U1700.6 (Vout)
- new net VDD: C1101.1, C1201.1, C1301.1, C1401.1, C1501.1, C1601.1, C1701.1, C1806.1, C1902.1, C5001.1, R1422.1, R1902.1, U1100.1 (VDD1), U1200.1 (VDD1), U1300.1 (VDD1), U1400.1 (VDD1), U1500.1 (VDD1), U1600.8 (VDD2), U1700.1 (VDD1), U1800.8 (VDD2), U1900.2 (VDD), U5001.1 (VDD1)
- no-connect marks 2 -> 3
Other:
- note added: "D"
- note added: "G"
- note added: "S"
- note added: "TruthTable\nVI Vled VO\nH OFF H\nL ON L"
- note removed: "The smartcard is powered by U500 GPIO"
- moved on the sheet: C1001, C1002, P1000, R1001
